File: 4_switch_array/4_switch_array.kicad_pcb (KiCad board)
At the start: 2 copper layers, 45.5 x 48.5 mm, 23 parts, among them J1 Conn_01x04, J2 Conn_01x04, J3 Conn_01x02, J4 Conn_01x02, J5 Conn_01x02, J6 Conn_01x02, J7 Conn_01x02, Q1 Q_NPN_EBC, Q2 Q_NPN_EBC, Q3 Q_NPN_EBC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

Commit message: Changed pinout to VCC-GND
Connections:
- J1 pad 2: Net-(J1-Pad2) -> GND
- J1 pad 3: Net-(J1-Pad3) -> SER_IN
- J1 pad 4: GND -> SRCLR
- J2 pad 2: Net-(J2-Pad2) -> GND
- J2 pad 3: Net-(J2-Pad3) -> RCLK
- J2 pad 4: GND -> SRCK
- J3 pad 1: GND -> Net-(J3-Pad1)
- J3 pad 2: Net-(J3-Pad2) -> GND
- J4 pad 1: GND -> Net-(J4-Pad1)
- J4 pad 2: Net-(J4-Pad2) -> GND
- J5 pad 1: GND -> Net-(J5-Pad1)
- J5 pad 2: Net-(J5-Pad2) -> GND
- J6 pad 1: GND -> Net-(J6-Pad1)
- J6 pad 2: Net-(J6-Pad2) -> GND
- Q1 pad 1: Net-(J3-Pad2) -> Net-(J3-Pad1)
- Q2 pad 1: Net-(J4-Pad2) -> Net-(J4-Pad1)
- Q3 pad 1: Net-(J5-Pad2) -> Net-(J5-Pad1)
- Q4 pad 1: Net-(J6-Pad2) -> Net-(J6-Pad1)
- U1 pad 12: Net-(J2-Pad1) -> RCLK
- U1 pad 13: Net-(J2-Pad2) -> SRCK
- U1 pad 3: Net-(J1-Pad1) -> SER_IN
- U1 pad 8: Net-(J1-Pad2) -> SRCLR
Routing:
- net RCLK: track 0.00 -> 33.3 mm
- net Net-(J2-Pad1): track 31.2 -> 0.00 mm
- net SRCK: track 0.00 -> 31.0 mm
- net Net-(J1-Pad2): track 30.7 -> 0.00 mm
- net Net-(J2-Pad2): track 28.9 -> 0.00 mm
- net SRCLR: track 0.00 -> 28.6 mm
- net Net-(J1-Pad1): track 18.5 -> 0.00 mm
- net SER_IN: track 0.00 -> 16.2 mm
- net Net-(J6-Pad2): track 11.2 -> 0.00 mm
- net Net-(J5-Pad2): track 11.2 -> 0.00 mm
- net Net-(J4-Pad1): track 0.00 -> 10.7 mm
- net Net-(J6-Pad1): track 0.00 -> 10.1 mm
- net Net-(J5-Pad1): track 0.00 -> 10.1 mm
- net Net-(J4-Pad2): track 9.62 -> 0.00 mm
- net Net-(J3-Pad1): track 0.00 -> 8.91 mm
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