File: power_supply/power_supply.kicad_pcb (KiCad board)
At the start: 2 copper layers, 45.5 x 30 mm, 14 parts, among them J1 Conn_01x04, J2 Conn_01x02, J3 Conn_01x02, U1 LM2596

Commit message: Changed pinout to VCC-GND
Connections:
- J1 pad 1: Net-(J1-Pad1) -> Net-(C1-Pad1)
- J1 pad 2: Net-(J1-Pad2) -> GND
- J1 pad 3: Net-(C1-Pad1) -> Net-(J1-Pad3)
- J1 pad 4: GND -> Net-(J1-Pad4)
- J2 pad 1: GND -> Net-(C2-Pad1)
- J2 pad 2: Net-(C2-Pad1) -> GND
- J3 pad 1: GND -> Net-(C2-Pad1)
Routing:
- net Net-(C2-Pad1): track 41.4 -> 40.1 mm
- net Net-(C1-Pad1): track 17.2 -> 18.2 mm
Changed lines of the file:
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@@
     (thickness 1.6)
     (drawings 17)
-    (tracks 19)
+    (tracks 21)
     (zones 0)
     (modules 14)
@@
   (net 3 "Net-(C2-Pad1)")
   (net 4 "Net-(D1-Pad1)")
-  (net 5 "Net-(J1-Pad1)")
-  (net 6 "Net-(J1-Pad2)")
+  (net 5 "Net-(J1-Pad4)")
+  (net 6 "Net-(J1-Pad3)")
   (net_class Default "This is the default net class."
     (clearance 0.2)
@@
     (add_net "Net-(C2-Pad1)")
     (add_net "Net-(D1-Pad1)")
-    (add_net "Net-(J1-Pad1)")
-    (add_net "Net-(J1-Pad2)")
+    (add_net "Net-(J1-Pad3)")
+    (add_net "Net-(J1-Pad4)")
   )
   (module Symbol:Symbol_CreativeCommons_SilkScreenTop_Type2_Small (layer F.Cu)
@@
     (fp_line (start -2.45 -2.35) (end -2.45 3.4) (layer F.Fab) (width 0.1))
     (pad 4 thru_hole oval (at 7.5 0 90) (size 1.7 1.95) (drill 0.95) (layers *.Cu *.Mask)
+      (net 5 "Net-(J1-Pad4)"))
+    (pad 3 thru_hole oval (at 5 0 90) (size 1.7 1.95) (drill 0.95) (layers *.Cu *.Mask)
+      (net 6 "Net-(J1-Pad3)"))
+    (pad 2 thru_hole oval (at 2.5 0 90) (size 1.7 1.95) (drill 0.95) (layers *.Cu *.Mask)
       (net 1 GND))
-    (pad 3 thru_hole oval (at 5 0 90) (size 1.7 1.95) (drill 0.95) (layers *.Cu *.Mask)
+    (pad 1 thru_hole roundrect (at 0 0 90) (size 1.7 1.95) (drill 0.95) (layers *.Cu *.Mask) (roundrect_rratio 0.147059)
       (net 2 "Net-(C1-Pad1)"))
-    (pad 2 thru_hole oval (at 2.5 0 90) (size 1.7 1.95) (drill 0.95) (layers *.Cu *.Mask)
-      (net 6 "Net-(J1-Pad2)"))
-    (pad 1 thru_hole roundrect (at 0 0 90) (size 1.7 1.95) (drill 0.95) (layers *.Cu *.Mask) (roundrect_rratio 0.147059)
-      (net 5 "Net-(J1-Pad1)"))
     (model ${KISYS3DMOD}/Connector_JST.3dshapes/JST_XH_B4B-XH-A_1x04_P2.50mm_Vertical.wrl
       (at (xyz 0 0 0))
@@
     (fp_line (start -2.45 -2.35) (end -2.45 3.4) (layer F.Fab) (width 0.1))
     (pad 2 thru_hole oval (at 2.5 0 180) (size 1.7 2) (drill 1) (layers *.Cu *.Mask)
+      (net 1 GND))
+    (pad 1 thru_hole roundrect (at 0 0 180) (size 1.7 2) (drill 1) (layers *.Cu *.Mask) (roundrect_rratio 0.147059)
       (net 3 "Net-(C2-Pad1)"))
-    (pad 1 thru_hole roundrect (at 0 0 180) (size 1.7 2) (drill 1) (layers *.Cu *.Mask) (roundrect_rratio 0.147059)
-      (net 1 GND))
     (model ${KISYS3DMOD}/Connector_JST.3dshapes/JST_XH_B2B-XH-A_1x02_P2.50mm_Vertical.wrl
       (at (xyz 0 0 0))
@@
     )
     (pad 1 thru_hole roundrect (at 0 0) (size 1.7 2) (drill 1) (layers *.Cu *.Mask) (roundrect_rratio 0.147059)
-      (net 1 GND))
+      (net 3 "Net-(C2-Pad1)"))
     (pad 2 thru_hole oval (at 2.5 0) (size 1.7 2) (drill 1) (layers *.Cu *.Mask)
       (net 3 "Net-(C2-Pad1)"))
@@
     (arrow2b (pts (xy 158.5 101.5) (xy 159.626504 100.913579)))
   )
-  (gr_text NC (at 168 130.5) (layer F.SilkS)
+  (gr_text NC (at 168 123) (layer F.SilkS)
     (effects (font (size 1 1) (thickness 0.15)))
   )
-  (gr_text NC (at 168 128) (layer F.SilkS)
+  (gr_text NC (at 168 125.5) (layer F.SilkS)
     (effects (font (size 1 1) (thickness 0.15)))
   )
-  (gr_text GND (at 168 123) (layer F.SilkS)
+  (gr_text GND (at 168 128) (layer F.SilkS)
     (effects (font (size 1 1) (thickness 0.15)))
   )
-  (gr_text VCC (at 168 125.5) (layer F.SilkS)
+  (gr_text VCC (at 168 130.5) (layer F.SilkS)
     (effects (font (size 1 1) (thickness 0.15)))
   )
-  (gr_text VCC (at 194 121) (layer F.SilkS)
+  (gr_text VCC (at 190.5 121) (layer F.SilkS)
     (effects (font (size 1 1) (thickness 0.15)))
   )
-  (gr_text GND (at 190.5 121) (layer F.SilkS)
+  (gr_text GND (at 194 121) (layer F.SilkS)
     (effects (font (size 1 1) (thickness 0.15)))
   )
-  (gr_text GND (at 194 133) (layer F.SilkS)
+  (gr_text GND (at 190.5 133) (layer F.SilkS)
     (effects (font (size 1 1) (thickness 0.15)))
   )
-  (gr_text VCC (at 190.5 133) (layer F.SilkS)
+  (gr_text VCC (at 194 133) (layer F.SilkS)
     (effects (font (size 1 1) (thickness 0.15)))
   )
@@
   (gr_line (start 204 142) (end 158.5 142) (layer Edge.Cuts) (width 0.05))
   (gr_line (start 158.5 142) (end 158.5 112) (layer Edge.Cuts) (width 0.05))
-  (segment (start 172.5 126.5) (end 172.5 128.5) (width 1.5) (layer F.Cu) (net 2))
-  (segment (start 171.5 125.5) (end 172.5 126.5) (width 1.5) (layer F.Cu) (net 2))
-  (segment (start 163 125.5) (end 171.5 125.5) (width 1.5) (layer F.Cu) (net 2))
-  (segment (start 171.5 124.5) (end 174.5 121.5) (width 1.5) (layer F.Cu) (net 2))
-  (segment (start 171.5 125.5) (end 171.5 124.5) (width 1.5) (layer F.Cu) (net 2))
-  (segment (start 191 127) (end 191 137.5) (width 1.5) (layer F.Cu) (net 3))
+  (segment (start 170.5 130.5) (end 172.5 128.5) (width 1.5) (layer F.Cu) (net 2))
+  (segment (start 163 130.5) (end 170.5 130.5) (width 1.5) (layer F.Cu) (net 2))
+  (segment (start 172.5 123.5) (end 174.5 121.5) (width 1.5) (layer F.Cu) (net 2))
+  (segment (start 172.5 128.5) (end 172.5 123.5) (width 1.5) (layer F.Cu) (net 2))
   (segment (start 191 127) (end 197 127) (width 1.5) (layer F.Cu) (net 3))
   (segment (start 191 125.302944) (end 191 127) (width 1.5) (layer F.Cu) (net 3))
   (segment (start 191 124.5) (end 191 125.302944) (width 1.5) (layer F.Cu) (net 3))
   (segment (start 179.6 117.3) (end 183.8 117.3) (width 1.5) (layer F.Cu) (net 3))
-  (segment (start 183.8 117.3) (end 191 124.5) (width 1.5) (layer F.Cu) (net 3))
-  (segment (start 193.5 118.5) (end 193.5 116.5) (width 1.5) (layer F.Cu) (net 3))
-  (segment (start 189.25 122.75) (end 193.5 118.5) (width 1.5) (layer F.Cu) (net 3))
+  (segment (start 190.094447 117.405553) (end 187 120.5) (width 1.5) (layer F.Cu) (net 3))
+  (segment (start 191 116.5) (end 190.094447 117.405553) (width 1.5) (layer F.Cu) (net 3))
+  (segment (start 183.8 117.3) (end 187 120.5) (width 1.5) (layer F.Cu) (net 3))
+  (segment (start 187 120.5) (end 191 124.5) (width 1.5) (layer F.Cu) (net 3))
+  (segment (start 191 127) (end 191 130.5) (width 1.5) (layer F.Cu) (net 3))
+  (segment (start 193.5 133) (end 193.5 137.5) (width 1.5) (layer F.Cu) (net 3))
+  (segment (start 191 130.5) (end 193.5 133) (width 1.5) (layer F.Cu) (net 3))
   (segment (start 186 135.2) (end 186 127) (width 1.5) (layer F.Cu) (net 4))
   (segment (start 186 137.5) (end 186 135.2) (width 1.5) (layer F.Cu) (net 4))
