File: hardware/12_24_boost_converter/12_24_boost_converter/12_24_boost_converter.sch (KiCad schematic (older format))
At the start: 14 parts, among them J1 Conn_01x02, J2 Conn_01x02, J3 Conn_01x02, Q1 IRFZ24NPBF, U1 LM555xM

Commit message: Update boost converter
Parts:
- added D2: LED, LED_THT:LED_D3.0mm, symbol Device:LED
- added R5: 560, Resistor_THT:R_Axial_DIN0411_L9.9mm_D3.6mm_P12.70mm_Horizontal, symbol Device:R_Small
- C1, C2: value 10nF -> 100nF
- R1, R2, R3: value 330 -> 47
Connections:
- net +12V: now also R5.2
- net GND: now also D2.1 (K)
- new net: D2.2 (A), R5.1
Changed lines of the file:
@@
 P 7550 4800
 F 0 "R2" V 7350 4800 50  0000 C CNN
-F 1 "330" V 7450 4800 50  0000 C CNN
+F 1 "47" V 7450 4800 50  0000 C CNN
 F 2 "Resistor_THT:R_Axial_DIN0411_L9.9mm_D3.6mm_P12.70mm_Horizontal" H 7550 4800 50  0001 C CNN
 F 3 "~" H 7550 4800 50  0001 C CNN
@@
 P 7550 4500
 F 0 "R1" V 7746 4500 50  0000 C CNN
-F 1 "330" V 7655 4500 50  0000 C CNN
+F 1 "47" V 7655 4500 50  0000 C CNN
 F 2 "Resistor_THT:R_Axial_DIN0411_L9.9mm_D3.6mm_P12.70mm_Horizontal" H 7550 4500 50  0001 C CNN
 F 3 "~" H 7550 4500 50  0001 C CNN
@@
 P 6200 5000
 F 0 "C2" H 6000 4950 50  0000 C CNN
-F 1 "10nF" H 6000 5050 50  0000 C CNN
+F 1 "100nF" H 6000 5050 50  0000 C CNN
 F 2 "Capacitor_THT:C_Disc_D5.1mm_W3.2mm_P5.00mm" H 6200 5000 50  0001 C CNN
 F 3 "~" H 6200 5000 50  0001 C CNN
@@
 P 5850 4700
 F 0 "C1" H 5650 4650 50  0000 C CNN
-F 1 "10nF" H 5650 4750 50  0000 C CNN
+F 1 "100nF" H 5650 4750 50  0000 C CNN
 F 2 "Capacitor_THT:C_Disc_D5.1mm_W3.2mm_P5.00mm" H 5850 4700 50  0001 C CNN
 F 3 "~" H 5850 4700 50  0001 C CNN
@@
 P 8150 4500
 F 0 "R3" V 8346 4500 50  0000 C CNN
-F 1 "330" V 8250 4500 50  0000 C CNN
+F 1 "47" V 8250 4500 50  0000 C CNN
 F 2 "Resistor_THT:R_Axial_DIN0411_L9.9mm_D3.6mm_P12.70mm_Horizontal" H 8150 4500 50  0001 C CNN
 F 3 "~" H 8150 4500 50  0001 C CNN
@@
 Wire Wire Line
 	6900 4250 7100 4250
+$Comp
+L Device:R_Small R5
+U 1 1 60AD3129
+P 11750 4250
+F 0 "R5" V 11946 4250 50  0000 C CNN
+F 1 "560" V 11850 4250 50  0000 C CNN
+F 2 "Resistor_THT:R_Axial_DIN0411_L9.9mm_D3.6mm_P12.70mm_Horizontal" H 11750 4250 50  0001 C CNN
+F 3 "~" H 11750 4250 50  0001 C CNN
+	1    11750 4250
+	1    0    0    1
+$EndComp
+$Comp
+L power:GND #PWR010
+U 1 1 60AD3CB0
+P 11750 5300
+F 0 "#PWR010" H 11750 5050 50  0001 C CNN
+F 1 "GND" H 11755 5127 50  0000 C CNN
+F 2 "" H 11750 5300 50  0001 C CNN
+F 3 "" H 11750 5300 50  0001 C CNN
+	1    11750 5300
+	1    0    0    -1
+$EndComp
+$Comp
+L power:+12V #PWR04
+U 1 1 60AD4445
+P 11750 3700
+F 0 "#PWR04" H 11750 3550 50  0001 C CNN
+F 1 "+12V" H 11765 3828 50  0000 L CNN
+F 2 "" H 11750 3700 50  0001 C CNN
+F 3 "" H 11750 3700 50  0001 C CNN
+	1    11750 3700
+	1    0    0    -1
+$EndComp
+$Comp
+L Device:LED D2
+U 1 1 60AD5387
+P 11750 4850
+F 0 "D2" V 11789 4732 50  0000 R CNN
+F 1 "LED" V 11698 4732 50  0000 R CNN
+F 2 "LED_THT:LED_D3.0mm" H 11750 4850 50  0001 C CNN
+F 3 "~" H 11750 4850 50  0001 C CNN
+	1    11750 4850
+	0    -1   -1   0
+$EndComp
+Wire Wire Line
+	11750 5300 11750 5000
+Wire Wire Line
+	11750 4700 11750 4350
+Wire Wire Line
+	11750 4150 11750 3700
 $EndSCHEMATC
