File: hardware/hub_PCB_redesign/beehive.sch (KiCad schematic (older format))
At the start: 28 parts, among them CON1 BARREL_JACK, J1 USB_A, P1 D1, P10 A2, P11 A3, P12 UART, P13 I2C 1, P14 I2C 2, P15 12V, P2 D2, P3 D3, P4 D4, P5 D5, P6 D6, P7 D7, P8 D8, P9 A1, U1 LM2596, U2 LM2596, U3 ESP32-DEVKITC-32D

Commit message: update main hub
Parts:
- removed U1, U2: LM2596, footprints:LM2596, symbol flypi_components:LM2596
- added U1, U2: LM2596T-5, Package_TO_SOT_THT:TO-220-5_P3.4x3.7mm_StaggerOdd_Lead3.8mm_Vertical, symbol Regulator_Switching:LM2596T-5
- U3: footprint MODULE_ESP32-DEVKITC-32D -> footprints:MODULE_ESP32-DEVKITC-32D; symbol ESP32-DEVKITC-32D:ESP32-DEVKITC-32D -> beehive-rescue:ESP32-DEVKITC-32D-ESP32-DEVKITC-32D
Connections:
- net +5V: now also P1.3 (Pin_3), P10.3 (Pin_3), P11.3 (Pin_3), P12.3 (Pin_3), P13.3 (Pin_3), P14.3 (Pin_3), P2.3 (Pin_3), P3.3 (Pin_3), P4.3 (Pin_3), P5.3 (Pin_3), P6.3 (Pin_3), P7.3 (Pin_3), P8.3 (Pin_3), P9.3 (Pin_3), U2.4 (FB); no longer P1.1 (Pin_1), P10.1 (Pin_1), P11.1 (Pin_1), P12.1 (Pin_1), P13.1 (Pin_1), P14.1 (Pin_1), P2.1 (Pin_1), P3.1 (Pin_1), P4.1 (Pin_1), P5.1 (Pin_1), P6.1 (Pin_1), P7.1 (Pin_1), P8.1 (Pin_1), P9.1 (Pin_1)
- net A1-3: now also P9.1 (Pin_1); no longer P9.3 (Pin_3)
- net A1-4: now also P9.2 (Pin_2); no longer P9.4 (Pin_4)
- net A2-3: now also P10.1 (Pin_1); no longer P10.3 (Pin_3)
- net A2-4: now also P10.2 (Pin_2); no longer P10.4 (Pin_4)
- net A3-3: now also P11.1 (Pin_1); no longer P11.3 (Pin_3)
- net A3-4: now also P11.2 (Pin_2); no longer P11.4 (Pin_4)
- net D1-3: now also P1.1 (Pin_1); no longer P1.3 (Pin_3)
- net D1-4: now also P1.2 (Pin_2); no longer P1.4 (Pin_4)
- net D2-3: now also P2.1 (Pin_1); no longer P2.3 (Pin_3)
- net D2-4: now also P2.2 (Pin_2); no longer P2.4 (Pin_4)
- net D3-3: now also P3.1 (Pin_1); no longer P3.3 (Pin_3)
- net D3-4: now also P3.2 (Pin_2); no longer P3.4 (Pin_4)
- net D4-3: now also P4.1 (Pin_1); no longer P4.3 (Pin_3)
- net D4-4: now also P4.2 (Pin_2); no longer P4.4 (Pin_4)
- net D5-3: now also P5.1 (Pin_1); no longer P5.3 (Pin_3)
- net D5-4: now also P5.2 (Pin_2); no longer P5.4 (Pin_4)
- net D6-3: now also P6.1 (Pin_1); no longer P6.3 (Pin_3)
- net D6-4: now also P6.2 (Pin_2); no longer P6.4 (Pin_4)
- net D7-3: now also P7.1 (Pin_1); no longer P7.3 (Pin_3)
- net D7-4: now also P7.2 (Pin_2); no longer P7.4 (Pin_4)
- net D8-3: now also P8.1 (Pin_1); no longer P8.3 (Pin_3)
- net D8-4: now also P8.2 (Pin_2); no longer P8.4 (Pin_4)
- net GND: now also P1.4 (Pin_4), P10.4 (Pin_4), P11.4 (Pin_4), P12.4 (Pin_4), P13.4 (Pin_4), P14.4 (Pin_4), P15.4 (Pin_4), P2.4 (Pin_4), P3.4 (Pin_4), P4.4 (Pin_4), P5.4 (Pin_4), P6.4 (Pin_4), P7.4 (Pin_4), P8.4 (Pin_4), P9.4 (Pin_4), U1.3 (GND), U1.5 (~ON~/OFF), U2.3 (GND), U2.5 (~ON~/OFF); no longer P1.2 (Pin_2), P10.2 (Pin_2), P11.2 (Pin_2), P12.2 (Pin_2), P13.2 (Pin_2), P14.2 (Pin_2), P15.2 (Pin_2), P2.2 (Pin_2), P3.2 (Pin_2), P4.2 (Pin_2), P5.2 (Pin_2), P6.2 (Pin_2), P7.2 (Pin_2), P8.2 (Pin_2), P9.2 (Pin_2)
- net I2C_1-3: now also P13.1 (Pin_1); no longer P13.3 (Pin_3)
- net I2C_1-4: now also P13.2 (Pin_2); no longer P13.4 (Pin_4)
- net I2C_2-3: now also P14.1 (Pin_1); no longer P14.3 (Pin_3)
- net I2C_2-4: now also P14.2 (Pin_2); no longer P14.4 (Pin_4)
- net RX: now also P12.2 (Pin_2); no longer P12.4 (Pin_4)
- net TX: now also P12.1 (Pin_1); no longer P12.3 (Pin_3)
- net at C1.1, C3.1, CON1.1: now also P15.3 (Pin_3), U1.1 (VIN), U2.1 (VIN); no longer P15.1 (Pin_1)
- net at D1.1 (K), L1.1: now also U1.2 (OUT)
- net at C2.1, J1.1 (VBUS), L1.2: now also U1.4 (FB)
- net at D2.1 (K), L2.1: now also U2.2 (OUT)
Other:
- note added: "DATA 1\n"
- note removed: "DATA 1"

Commit message: Update on 12V5A system power line
- 12V5A power line is now represented by two connectors with 2 pins across all the modules
- all .png previews are updated. The central hub now has previews for schematics, PCB tracing and 3D model
- peltier module now has two 12V5A connectors with redesigned one side of the bridge. Now all MOSFETs can be equipped with heatsinks
- hum/temp sensor now has its connector position reversed to mimic Grove's one
- hum/temp and gas sensors now have a small BeeHive logo on front layer rather than one big on back layer
- hum/temp sensor now use only one layer for signals and one layer for ground
- switch arrays now have two connectors for 12V5A and 5V3A power lines
- switch arrays had their power lines better traced (no sharp turns)
- power supply (12V5A to 5V3A) now has two connectors for 12V5A power line
- one trace of power supply, which lies in between LM2596's legs, was narrowed to ensure that it will not be accidentally soldered or damaged during placement
Parts:
- removed P15: 12V, Connector_JST:JST_XH_B04B-XH-A_04x2.50mm_Straight, symbol Connector_Generic:Conn_01x04
- added P15, P16: Conn_01x02, Connector_JST:JST_XH_B2B-XH-A_1x02_P2.50mm_Vertical, symbol Connector_Generic:Conn_01x02
Connections:
- net GND: now also P15.2 (Pin_2), P16.2 (Pin_2)
- net at C1.1, C3.1, CON1.1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: now also P15.1 (Pin_1), P16.1 (Pin_1)
- no-connect marks 10 -> 8
Other:
- note added: "12V line"
Changed lines of the file:
@@
 Wire Notes Line
 	5600 7600 5600 6550
-Text Notes 1850 5450 0    100  ~ 0
-To additional\nPS 5V3A
 Text Notes 800  1850 0    100  ~ 0
 12V5A
-NoConn ~ 2300 5700
-NoConn ~ 2300 5800
 Wire Notes Line
 	2950 6250 1750 6250
@@
 $EndComp
 $Comp
-L Connector_Generic:Conn_01x04 P15
-U 1 1 5E555C9B
-P 2500 5800
-F 0 "P15" H 2500 6050 50  0000 C CNN
-F 1 "12V" V 2600 5750 50  0000 C CNN
-F 2 "Connector_JST:JST_XH_B04B-XH-A_04x2.50mm_Straight" H 2500 5800 50  0001 C CNN
-F 3 "" H 2500 5800 50  0000 C CNN
-	1    2500 5800
-	1    0    0    -1
-$EndComp
-$Comp
 L Connector_Generic:Conn_01x04 P14
 U 1 1 5E34A2F6
@@
 	1550 5900 2300 5900
 Wire Wire Line
-	1550 3900 1550 5900
+	1550 3900 1550 5600
 Wire Wire Line
 	6050 7350 6450 7350
@@
 Wire Wire Line
 	3150 4450 4050 4450
+$Comp
+L Connector_Generic:Conn_01x02 P16
+U 1 1 5FD3103D
+P 2500 5900
+F 0 "P16" H 2580 5846 50  0000 L CNN
+F 1 "Conn_01x02" H 2580 5801 50  0001 L CNN
+F 2 "Connector_JST:JST_XH_B2B-XH-A_1x02_P2.50mm_Vertical" H 2500 5900 50  0001 C CNN
+F 3 "~" H 2500 5900 50  0001 C CNN
+	1    2500 5900
+	1    0    0    -1
+$EndComp
+Wire Wire Line
+	2300 5600 1550 5600
+Connection ~ 1550 5600
+Wire Wire Line
+	1550 5600 1550 5900
+Wire Wire Line
+	2100 6000 2100 5700
+Wire Wire Line
+	2100 5700 2300 5700
+Connection ~ 2100 6000
+$Comp
+L Connector_Generic:Conn_01x02 P15
+U 1 1 5FD3163B
+P 2500 5600
+F 0 "P15" H 2580 5546 50  0000 L CNN
+F 1 "Conn_01x02" H 2580 5501 50  0001 L CNN
+F 2 "Connector_JST:JST_XH_B2B-XH-A_1x02_P2.50mm_Vertical" H 2500 5600 50  0001 C CNN
+F 3 "~" H 2500 5600 50  0001 C CNN
+	1    2500 5600
+	1    0    0    -1
+$EndComp
+Text Notes 1850 5450 0    100  ~ 0
+To additional\nPS 5V3A
+Text Notes 2850 5950 1    50   ~ 0
+12V line
 $EndSCHEMATC

Commit message: Add ESP32 5V trace and minor changes
ESP32 is now connected to the same line as Raspberry Pi that should reduce the noise.
Add new screenshot to the temperature breakout board

Co-Authored-By: Andre Maia Chagas <a.maia-chagas@sussex.ac.uk>
Connections:
- net +5V: no longer U3.19 (EXT_5V)
- net ESP_pow: now reaches C2.1, J1.1 (VBUS), L1.2, U1.4 (FB)
- net ESP_pow: now also U3.19 (EXT_5V)
Changed lines of the file:
@@
 Wire Wire Line
 	3950 3450 4050 3450
-Connection ~ 4050 3450
 Connection ~ 6500 1950
 $Comp
@@
 Wire Wire Line
 	6500 5350 7450 5350
-$Comp
-L power:+5V #PWR0111
-U 1 1 5E230612
-P 10300 1950
-F 0 "#PWR0111" H 10300 1800 50  0001 C CNN
-F 1 "+5V" V 10300 2150 50  0000 C CNN
-F 2 "" H 10300 1950 50  0001 C CNN
-F 3 "" H 10300 1950 50  0001 C CNN
-	1    10300 1950
-	0    1    -1   0
-$EndComp
 Wire Wire Line
 	7450 5350 7450 5300
@@
 	10850 3100 10850 2450
 Wire Wire Line
-	10300 1950 10200 1950
+	10350 1950 10200 1950
 Wire Wire Line
 	10850 2450 10200 2450
@@
 Wire Notes Line
 	1750 4700 4700 4700
-Wire Wire Line
-	4050 3450 4250 3450
-$Comp
-L power:+5V #PWR0104
-U 1 1 5EBCB95D
-P 4250 3450
-F 0 "#PWR0104" H 4250 3300 50  0001 C CNN
-F 1 "+5V" V 4265 3578 50  0000 L CNN
-F 2 "" H 4250 3450 50  0001 C CNN
-F 3 "" H 4250 3450 50  0001 C CNN
-	1    4250 3450
-	0    1    1    0
-$EndComp
 Wire Notes Line
 	4700 3150 4700 4700
@@
 Text Notes 2850 5950 1    50   ~ 0
 12V line
+$Comp
+L power:+5V #PWR0104
+U 1 1 5EBCB95D
+P 4250 3450
+F 0 "#PWR0104" H 4250 3300 50  0001 C CNN
+F 1 "+5V" V 4265 3578 50  0000 L CNN
+F 2 "" H 4250 3450 50  0001 C CNN
+F 3 "" H 4250 3450 50  0001 C CNN
+	1    4250 3450
+	0    1    1    0
+$EndComp
+Connection ~ 4050 3450
+Wire Wire Line
+	4050 3450 4250 3450
+Text GLabel 4100 1850 1    50   Input ~ 0
+ESP_pow
+Wire Wire Line
+	4100 1950 4100 1850
+Connection ~ 4100 1950
+Text GLabel 10350 1950 2    50   Input ~ 0
+ESP_pow
 $EndSCHEMATC
