File: hardware/4_switch_array_(ver 4)/4_switch_array.kicad_pcb (KiCad board)
At the start: 2 copper layers, 45.5 x 48.5 mm, 22 parts, among them J1 Conn_01x04, J2 Conn_01x04, J3 Conn_01x02, J4 Conn_01x02, J5 Conn_01x02, J6 Conn_01x02, J7 Conn_01x02, J8 Conn_01x02, Q1 Q_NPN_EBC, Q2 Q_NPN_EBC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

Commit message: Apply CERN-W license
Apply CERN-W license to all boards, move the first iteration of the IR_sensor to the archive

Co-Authored-By: Andre Maia Chagas <a.maia-chagas@sussex.ac.uk>
Other:
- board text added: "board by Ihor Sobianin licensed under CERN-OHL-W 2.0 https://ohwr.org/project/cernohl"
Changed lines of the file:
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@@
-(kicad_pcb (version 20171130) (host pcbnew "(5.1.7)-1")
+(kicad_pcb (version 20171130) (host pcbnew "(5.1.10)-1")
   (general
     (thickness 1.6)
-    (drawings 54)
+    (drawings 55)
     (tracks 50)
     (zones 0)
@@
     (visible_elements 7FFFFF7F)
     (pcbplotparams
-      (layerselection 0x00020_7ffffffe)
+      (layerselection 0x00030_7ffffffe)
       (usegerberextensions false)
       (usegerberattributes false)
@@
     )
   )
+  (gr_text "board by Ihor Sobianin\nlicensed under\nCERN-OHL-W 2.0\nhttps://ohwr.org/project/cernohl" (at 132.08 46.99) (layer F.SilkS)
+    (effects (font (size 0.5 0.5) (thickness 0.1)))
+  )
   (gr_text S0 (at 138.5 43.5 90) (layer F.SilkS)
