File: hardware/12V5A_breakout/12V5A_breakout.kicad_pcb (KiCad board)
At the start: 2 copper layers, 48.5 x 45.5 mm, 18 parts, among them J1 Barrel_Jack_Switch, J10 Conn_01x02, J2 Conn_01x02, J3 Conn_01x02, J4 Conn_01x02, J5 Conn_01x02, J6 Conn_01x02, J7 Conn_01x02, J8 Conn_01x02, J9 Conn_01x02

Commit message: Update 12V5A_breakout.kicad_pcb
Parts:
- moved J2 0.50 mm to (99.0, 51.0)
- moved J3 0.50 mm to (99.0, 61.0)
- moved J4 0.50 mm to (99.0, 71.0)
Changed lines of the file:
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@@
     (solder_mask_min_width 0.25)
     (aux_axis_origin 0 0)
-    (visible_elements FFFFFF7F)
+    (visible_elements 7FFFFFFF)
     (pcbplotparams
       (layerselection 0x3ffff_ffffffff)
@@
   )
   (module Connector_JST:JST_XH_B2B-XH-A_1x02_P2.50mm_Vertical (layer F.Cu)
-    (at 98.5 71 270)
+    (at 99 71 270)
     (descr "JST XH series connector, B2B-XH-A (http://www.jst-mfg.com/product/pdf/eng/eXH.pdf), generated with kicad-footprint-generator")
     (tags "connector JST XH vertical")
@@
   )
   (module Connector_JST:JST_XH_B2B-XH-A_1x02_P2.50mm_Vertical (layer F.Cu)
-    (at 98.5 61 270)
+    (at 99 61 270)
     (descr "JST XH series connector, B2B-XH-A (http://www.jst-mfg.com/product/pdf/eng/eXH.pdf), generated with kicad-footprint-generator")
     (tags "connector JST XH vertical")
@@
   )
   (module Connector_JST:JST_XH_B2B-XH-A_1x02_P2.50mm_Vertical (layer F.Cu)
-    (at 98.5 51 270)
+    (at 99 51 270)
     (descr "JST XH series connector, B2B-XH-A (http://www.jst-mfg.com/product/pdf/eng/eXH.pdf), generated with kicad-footprint-generator")
     (tags "connector JST XH vertical")
@@
     (effects (font (size 1 1) (thickness 0.15)))
   )
-  (gr_text 12V (at 102 64 90) (layer F.SilkS)
-    (effects (font (size 1 1) (thickness 0.15)))
-  )
-  (gr_text GND (at 102 60.5 90) (layer F.SilkS)
-    (effects (font (size 1 1) (thickness 0.15)))
-  )
-  (gr_text 12V (at 102 74 90) (layer F.SilkS)
-    (effects (font (size 1 1) (thickness 0.15)))
-  )
-  (gr_text GND (at 102 70.5 90) (layer F.SilkS)
+  (gr_text 12V (at 102.5 64 90) (layer F.SilkS)
+    (effects (font (size 1 1) (thickness 0.15)))
+  )
+  (gr_text GND (at 102.5 60.5 90) (layer F.SilkS)
+    (effects (font (size 1 1) (thickness 0.15)))
+  )
+  (gr_text 12V (at 102.5 74 90) (layer F.SilkS)
+    (effects (font (size 1 1) (thickness 0.15)))
+  )
+  (gr_text GND (at 102.5 70.5 90) (layer F.SilkS)
     (effects (font (size 1 1) (thickness 0.15)))
   )
@@
     (effects (font (size 1 1) (thickness 0.15)))
   )
-  (gr_text 12V (at 102 54 90) (layer F.SilkS)
-    (effects (font (size 1 1) (thickness 0.15)))
-  )
-  (gr_text GND (at 102 50.5 90) (layer F.SilkS)
+  (gr_text 12V (at 102.5 54 90) (layer F.SilkS)
+    (effects (font (size 1 1) (thickness 0.15)))
+  )
+  (gr_text GND (at 102.5 50.5 90) (layer F.SilkS)
     (effects (font (size 1 1) (thickness 0.15)))
   )
@@
   (segment (start 90 50.5) (end 97.5 43) (width 1.5) (layer F.Cu) (net 2))
   (segment (start 90 52.5) (end 90 50.5) (width 1.5) (layer F.Cu) (net 2))
-  (segment (start 93 53.5) (end 98.5 53.5) (width 1.5) (layer F.Cu) (net 2))
-  (segment (start 98.5 53.5) (end 109 53.5) (width 1.5) (layer F.Cu) (net 2))
   (segment (start 109 53.5) (end 119 53.5) (width 1.5) (layer F.Cu) (net 2))
-  (segment (start 98.5 73.5) (end 109 73.5) (width 1.5) (layer F.Cu) (net 2))
   (segment (start 109 73.5) (end 119 73.5) (width 1.5) (layer F.Cu) (net 2))
-  (segment (start 98.5 63.5) (end 93 63.5) (width 1.5) (layer F.Cu) (net 2))
   (segment (start 93 53.5) (end 93 63.5) (width 1.5) (layer F.Cu) (net 2))
-  (segment (start 98.5 63.5) (end 109 63.5) (width 1.5) (layer F.Cu) (net 2))
   (segment (start 109 63.5) (end 119 63.5) (width 1.5) (layer F.Cu) (net 2))
-  (segment (start 96 73.5) (end 98.5 73.5) (width 1.5) (layer F.Cu) (net 2))
+  (segment (start 92 52.5) (end 90 52.5) (width 1.25) (layer F.Cu) (net 2))
+  (segment (start 93 53.5) (end 92 52.5) (width 1.25) (layer F.Cu) (net 2))
+  (segment (start 99 63.5) (end 93 63.5) (width 1.5) (layer F.Cu) (net 2))
+  (segment (start 99 63.5) (end 109 63.5) (width 1.5) (layer F.Cu) (net 2))
+  (segment (start 96 73.5) (end 99 73.5) (width 1.5) (layer F.Cu) (net 2))
   (segment (start 93 63.5) (end 93 70.5) (width 1.5) (layer F.Cu) (net 2))
   (segment (start 93 70.5) (end 96 73.5) (width 1.5) (layer F.Cu) (net 2))
-  (segment (start 92 52.5) (end 90 52.5) (width 1.25) (layer F.Cu) (net 2))
-  (segment (start 93 53.5) (end 92 52.5) (width 1.25) (layer F.Cu) (net 2))
+  (segment (start 99 73.5) (end 109 73.5) (width 1.5) (layer F.Cu) (net 2))
+  (segment (start 99 53.5) (end 109 53.5) (width 1.5) (layer F.Cu) (net 2))
+  (segment (start 93 53.5) (end 99 53.5) (width 1.5) (layer F.Cu) (net 2))
   (segment (start 93 43) (end 88.04 43) (width 1) (layer F.Cu) (net 3))
   (zone (net 1) (net_name GND) (layer B.Cu) (hatch edge 0.508)

Commit message: Add version number to boards
Add version number to boards and update screenshots, zip gerber archives
Other:
- rule pad_to_mask_clearance: 0.051 -> 0
- board text added: "12V5A breakout v0.1"
- board text removed: "12V5A breakout"

Commit message: Apply CERN-W license
Apply CERN-W license to all boards, move the first iteration of the IR_sensor to the archive

Co-Authored-By: Andre Maia Chagas <a.maia-chagas@sussex.ac.uk>
Other:
- board text added: "board by Ihor Sobianin licensed under CERN-OHL-W 2.0 https://ohwr.org/project/cernohl"
Changed lines of the file:
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@@
-(kicad_pcb (version 20171130) (host pcbnew "(5.1.7)-1")
+(kicad_pcb (version 20171130) (host pcbnew "(5.1.10)-1")
   (general
     (thickness 1.6)
-    (drawings 28)
+    (drawings 29)
     (tracks 23)
     (zones 0)
@@
     (visible_elements 7FFFFFFF)
     (pcbplotparams
-      (layerselection 0x00020_7ffffffe)
+      (layerselection 0x00030_7ffffffe)
       (usegerberextensions false)
       (usegerberattributes false)
@@
     )
   )
+  (gr_text "board by Ihor Sobianin\nlicensed under\nCERN-OHL-W 2.0\nhttps://ohwr.org/project/cernohl" (at 78.74 53.34 90) (layer F.SilkS)
+    (effects (font (size 0.5 0.5) (thickness 0.1)))
+  )
   (gr_text 12V (at 112.5 64 90) (layer F.SilkS)

Commit message: boards review
Other:
- board text added: "12V5A breakout v0.2"
- board text removed: "12V5A breakout v0.1"
Changed lines of the file:
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@@
-(kicad_pcb (version 20171130) (host pcbnew "(5.1.10)-1")
+(kicad_pcb (version 20171130) (host pcbnew 5.1.10-88a1d61d58~90~ubuntu20.04.1)
   (general
     (thickness 1.6)
@@
     (visible_elements 7FFFFFFF)
     (pcbplotparams
-      (layerselection 0x00030_7ffffffe)
+      (layerselection 0x3ffff_ffffffff)
       (usegerberextensions false)
       (usegerberattributes false)
@@
     (pad 2 thru_hole oval (at 2.5 0 270) (size 1.7 2) (drill 1) (layers *.Cu *.Mask)
       (net 2 +12V))
-    (pad 1 thru_hole roundrect (at 0 0 270) (size 1.7 2) (drill 1) (layers *.Cu *.Mask) (roundrect_rratio 0.147059)
+    (pad 1 thru_hole roundrect (at 0 0 270) (size 1.7 2) (drill 1) (layers *.Cu *.Mask) (roundrect_rratio 0.1470588235294118)
       (net 1 GND))
     (model ${KISYS3DMOD}/Connector_JST.3dshapes/JST_XH_B2B-XH-A_1x02_P2.50mm_Vertical.wrl
@@
     (pad 2 thru_hole oval (at 2.5 0 270) (size 1.7 2) (drill 1) (layers *.Cu *.Mask)
       (net 2 +12V))
-    (pad 1 thru_hole roundrect (at 0 0 270) (size 1.7 2) (drill 1) (layers *.Cu *.Mask) (roundrect_rratio 0.147059)
+    (pad 1 thru_hole roundrect (at 0 0 270) (size 1.7 2) (drill 1) (layers *.Cu *.Mask) (roundrect_rratio 0.1470588235294118)
       (net 1 GND))
     (model ${KISYS3DMOD}/Connector_JST.3dshapes/JST_XH_B2B-XH-A_1x02_P2.50mm_Vertical.wrl
@@
     (pad 2 thru_hole oval (at 2.5 0 270) (size 1.7 2) (drill 1) (layers *.Cu *.Mask)
       (net 2 +12V))
-    (pad 1 thru_hole roundrect (at 0 0 270) (size 1.7 2) (drill 1) (layers *.Cu *.Mask) (roundrect_rratio 0.147059)
+    (pad 1 thru_hole roundrect (at 0 0 270) (size 1.7 2) (drill 1) (layers *.Cu *.Mask) (roundrect_rratio 0.1470588235294118)
       (net 1 GND))
     (model ${KISYS3DMOD}/Connector_JST.3dshapes/JST_XH_B2B-XH-A_1x02_P2.50mm_Vertical.wrl
@@
     (pad 2 thru_hole oval (at 2.5 0 270) (size 1.7 2) (drill 1) (layers *.Cu *.Mask)
       (net 2 +12V))
-    (pad 1 thru_hole roundrect (at 0 0 270) (size 1.7 2) (drill 1) (layers *.Cu *.Mask) (roundrect_rratio 0.147059)
+    (pad 1 thru_hole roundrect (at 0 0 270) (size 1.7 2) (drill 1) (layers *.Cu *.Mask) (roundrect_rratio 0.1470588235294118)
       (net 1 GND))
     (model ${KISYS3DMOD}/Connector_JST.3dshapes/JST_XH_B2B-XH-A_1x02_P2.50mm_Vertical.wrl
@@
     (pad 2 thru_hole oval (at 2.5 0 270) (size 1.7 2) (drill 1) (layers *.Cu *.Mask)
       (net 2 +12V))
-    (pad 1 thru_hole roundrect (at 0 0 270) (size 1.7 2) (drill 1) (layers *.Cu *.Mask) (roundrect_rratio 0.147059)
+    (pad 1 thru_hole roundrect (at 0 0 270) (size 1.7 2) (drill 1) (layers *.Cu *.Mask) (roundrect_rratio 0.1470588235294118)
       (net 1 GND))
     (model ${KISYS3DMOD}/Connector_JST.3dshapes/JST_XH_B2B-XH-A_1x02_P2.50mm_Vertical.wrl
@@
     (pad 2 thru_hole oval (at 2.5 0 270) (size 1.7 2) (drill 1) (layers *.Cu *.Mask)
       (net 2 +12V))
-    (pad 1 thru_hole roundrect (at 0 0 270) (size 1.7 2) (drill 1) (layers *.Cu *.Mask) (roundrect_rratio 0.147059)
+    (pad 1 thru_hole roundrect (at 0 0 270) (size 1.7 2) (drill 1) (layers *.Cu *.Mask) (roundrect_rratio 0.1470588235294118)
       (net 1 GND))
     (model ${KISYS3DMOD}/Connector_JST.3dshapes/JST_XH_B2B-XH-A_1x02_P2.50mm_Vertical.wrl
@@
     (pad 2 thru_hole oval (at 2.5 0 270) (size 1.7 2) (drill 1) (layers *.Cu *.Mask)
       (net 2 +12V))
-    (pad 1 thru_hole roundrect (at 0 0 270) (size 1.7 2) (drill 1) (layers *.Cu *.Mask) (roundrect_rratio 0.147059)
+    (pad 1 thru_hole roundrect (at 0 0 270) (size 1.7 2) (drill 1) (layers *.Cu *.Mask) (roundrect_rratio 0.1470588235294118)
       (net 1 GND))
     (model ${KISYS3DMOD}/Connector_JST.3dshapes/JST_XH_B2B-XH-A_1x02_P2.50mm_Vertical.wrl
@@
     (pad 2 thru_hole oval (at 2.5 0 270) (size 1.7 2) (drill 1) (layers *.Cu *.Mask)
       (net 2 +12V))
-    (pad 1 thru_hole roundrect (at 0 0 270) (size 1.7 2) (drill 1) (layers *.Cu *.Mask) (roundrect_rratio 0.147059)
+    (pad 1 thru_hole roundrect (at 0 0 270) (size 1.7 2) (drill 1) (layers *.Cu *.Mask) (roundrect_rratio 0.1470588235294118)
       (net 1 GND))
     (model ${KISYS3DMOD}/Connector_JST.3dshapes/JST_XH_B2B-XH-A_1x02_P2.50mm_Vertical.wrl
@@
     (pad 2 thru_hole oval (at 2.5 0 270) (size 1.7 2) (drill 1) (layers *.Cu *.Mask)
       (net 2 +12V))
-    (pad 1 thru_hole roundrect (at 0 0 270) (size 1.7 2) (drill 1) (layers *.Cu *.Mask) (roundrect_rratio 0.147059)
+    (pad 1 thru_hole roundrect (at 0 0 270) (size 1.7 2) (drill 1) (layers *.Cu *.Mask) (roundrect_rratio 0.1470588235294118)
       (net 1 GND))
     (model ${KISYS3DMOD}/Connector_JST.3dshapes/JST_XH_B2B-XH-A_1x02_P2.50mm_Vertical.wrl
@@
     (effects (font (size 1.25 1.25) (thickness 0.25)))
   )
-  (gr_text "12V5A breakout v0.1" (at 105.5 81) (layer F.SilkS)
+  (gr_text "12V5A breakout v0.2" (at 105.5 81) (layer F.SilkS)
     (effects (font (size 1.25 1.25) (thickness 0.25)))
   )
@@
       )
     )
+  )
+  (zone (net 0) (net_name "") (layers F&B.Cu) (hatch edge 0.508)
+    (connect_pads (clearance 0.5))
+    (min_thickness 0.254)
+    (keepout (tracks not_allowed) (vias not_allowed) (copperpour not_allowed))
+    (fill (arc_segments 32) (thermal_gap 0.508) (thermal_bridge_width 0.508))
+    (polygon
+      (pts
+        (xy 81.915 46.482) (xy 75.311 46.482) (xy 75.311 39.878) (xy 81.915 39.878)
+      )
+    )
+  )
+  (zone (net 0) (net_name "") (layers F&B.Cu) (hatch edge 0.508)
+    (connect_pads (clearance 0.5))
+    (min_thickness 0.254)
+    (keepout (tracks not_allowed) (vias not_allowed) (copperpour not_allowed))
+    (fill (arc_segments 32) (thermal_gap 0.508) (thermal_bridge_width 0.508))
+    (polygon
+      (pts
+        (xy 81.915 84.709) (xy 75.311 84.709) (xy 75.311 78.105) (xy 81.915 78.105)
+      )
+    )
+  )
+  (zone (net 0) (net_name "") (layers F&B.Cu) (hatch edge 0.508)
+    (connect_pads (clearance 0.5))
+    (min_thickness 0.254)
+    (keepout (tracks not_allowed) (vias not_allowed) (copperpour not_allowed))
+    (fill (arc_segments 32) (thermal_gap 0.508) (thermal_bridge_width 0.508))
+    (polygon
+      (pts
+        (xy 123.317 84.836) (xy 116.713 84.836) (xy 116.713 78.232) (xy 123.317 78.232)
+      )
+    )
+  )
+  (zone (net 0) (net_name "") (layers F&B.Cu) (hatch edge 0.508)
+    (connect_pads (clearance 0.5))
+    (min_thickness 0.254)
+    (keepout (tracks not_allowed) (vias not_allowed) (copperpour not_allowed))
+    (fill (arc_segments 32) (thermal_gap 0.508) (thermal_bridge_width 0.508))
+    (polygon
+      (pts
+        (xy 123.317 46.355) (xy 116.713 46.355) (xy 116.713 39.751) (xy 123.317 39.751)
+      )
+    )
