File: hardware/hum_temp_sensor/hum_temp_sensor.kicad_pcb (KiCad board)
At the start: 2 copper layers, 48.5 x 27.5 mm, 12 parts, among them J1 Conn_01x04, U1 DHT11

Commit message: update temp/humid sensor
Connections:
- J1 pad 1: +5V -> Net-(J1-Pad1)
- J1 pad 2: GND -> Net-(J1-Pad2)
- J1 pad 3: Net-(J1-Pad3) -> +5V
- J1 pad 4: Net-(J1-Pad4) -> GND
- R1 pad 2: Net-(J1-Pad4) -> Net-(J1-Pad1)
- U1 pad 2: Net-(J1-Pad4) -> Net-(J1-Pad1)
Routing:
- net Net-(J1-Pad1): track 0.00 -> 29.8 mm
- net Net-(J1-Pad4): track 23.2 -> 0.00 mm
- net +5V: track 48.4 -> 51.2 mm

Commit message: Update silk layer
Routing:
- net Net-(J1-Pad1): track 29.8 -> 28.4 mm
- net +5V: track 51.2 -> 50.4 mm

Commit message: Update on 12V5A system power line
- 12V5A power line is now represented by two connectors with 2 pins across all the modules
- all .png previews are updated. The central hub now has previews for schematics, PCB tracing and 3D model
- peltier module now has two 12V5A connectors with redesigned one side of the bridge. Now all MOSFETs can be equipped with heatsinks
- hum/temp sensor now has its connector position reversed to mimic Grove's one
- hum/temp and gas sensors now have a small BeeHive logo on front layer rather than one big on back layer
- hum/temp sensor now use only one layer for signals and one layer for ground
- switch arrays now have two connectors for 12V5A and 5V3A power lines
- switch arrays had their power lines better traced (no sharp turns)
- power supply (12V5A to 5V3A) now has two connectors for 12V5A power line
- one trace of power supply, which lies in between LM2596's legs, was narrowed to ensure that it will not be accidentally soldered or damaged during placement
Parts:
- removed the G*** at (122.5, 109.5)
- added G***: LOGO, logo-beehive:logo-beehive-7_2х6_7mm, F.Cu at (98.0, 119.0)
- moved J1 7.57 mm to (129.5, 113.0), turned to 90 degrees
- moved REF** 4.50 mm to (106.5, 119.5)
Routing:
- net Net-(J1-Pad1): track 28.4 -> 26.4 mm
Other:
- rule pad_to_mask_clearance: 0.051 -> 0
- board text added: "Connector is placed this way to be compateble with Grove module"

Commit message: Add version number to boards
Add version number to boards and update screenshots, zip gerber archives
Other:
- board text added: "Humidity & temperature sensor v0.1"
- board text removed: "Humidity & temperature sensor for BeeHive"

Commit message: Apply CERN-W license
Apply CERN-W license to all boards, move the first iteration of the IR_sensor to the archive

Co-Authored-By: Andre Maia Chagas <a.maia-chagas@sussex.ac.uk>
Other:
- board text added: "board by Ihor Sobianin licensed under CERN-OHL-W 2.0 https://ohwr.org/project/cernohl"

Commit message: boards review
Parts:
- R2: value 1k -> 220
Other:
- board text added: "Humidity & temperature sensor v0.2"
- board text removed: "Humidity & temperature sensor v0.1"
