File: hardware/hum_temp_sensor/hum_temp_sensor.sch (KiCad schematic (older format))
At the start: 6 parts, among them J1 Conn_01x04, U1 DHT11

Commit message: update temp/humid sensor
Connections:
- net +5V: now also J1.3 (Pin_3); no longer J1.1 (Pin_1)
- net GND: now also J1.4 (Pin_4); no longer J1.2 (Pin_2)
- net at R1.2, U1.2 (IO): now also J1.1 (Pin_1); no longer J1.4 (Pin_4)
Other:
- moved on the sheet: C1
Changed lines of the file:
@@
 	1    0    0    -1
 $EndComp
-Wire Wire Line
-	2650 2100 2900 2100
-Wire Wire Line
-	2900 2100 2900 2650
-Wire Wire Line
-	3100 2000 3100 1700
 $Comp
 L power:GND #PWR05
 U 1 1 5F3421BF
-P 4250 2650
-F 0 "#PWR05" H 4250 2400 50  0001 C CNN
-F 1 "GND" H 4255 2477 50  0000 C CNN
-F 2 "" H 4250 2650 50  0001 C CNN
-F 3 "" H 4250 2650 50  0001 C CNN
-	1    4250 2650
-	1    0    0    -1
+P 4250 2150
+F 0 "#PWR05" H 4250 1900 50  0001 C CNN
+F 1 "GND" H 4255 1977 50  0000 C CNN
+F 2 "" H 4250 2150 50  0001 C CNN
+F 3 "" H 4250 2150 50  0001 C CNN
+	1    4250 2150
+	0    1    1    0
 $EndComp
 Wire Wire Line
 	4300 2150 4250 2150
-Wire Wire Line
-	4250 2150 4250 2650
-Wire Wire Line
-	2650 2300 3350 2300
 Wire Wire Line
 	3650 2300 3650 2550
@@
 	-1   0    0    -1
 $EndComp
-NoConn ~ 2650 2200
+NoConn ~ 2650 2100
 $Comp
 L power:+5V #PWR06
@@
 Wire Wire Line
 	3350 2300 3650 2300
-Wire Wire Line
-	2650 2000 3100 2000
 $Comp
 L Device:C C1
 U 1 1 5F345169
-P 3100 2500
-F 0 "C1" H 3215 2546 50  0000 L CNN
-F 1 "100nF" H 3215 2455 50  0000 L CNN
-F 2 "Capacitor_THT:C_Disc_D7.0mm_W2.5mm_P5.00mm" H 3138 2350 50  0001 C CNN
-F 3 "~" H 3100 2500 50  0001 C CNN
-	1    3100 2500
+P 3100 2700
+F 0 "C1" H 3215 2746 50  0000 L CNN
+F 1 "100nF" H 3215 2655 50  0000 L CNN
+F 2 "Capacitor_THT:C_Disc_D7.0mm_W2.5mm_P5.00mm" H 3138 2550 50  0001 C CNN
+F 3 "~" H 3100 2700 50  0001 C CNN
+	1    3100 2700
 	1    0    0    -1
 $EndComp
@@
 L power:GND #PWR03
 U 1 1 5F3459C1
-P 3100 2650
-F 0 "#PWR03" H 3100 2400 50  0001 C CNN
-F 1 "GND" H 3105 2477 50  0000 C CNN
-F 2 "" H 3100 2650 50  0001 C CNN
-F 3 "" H 3100 2650 50  0001 C CNN
-	1    3100 2650
+P 3100 2850
+F 0 "#PWR03" H 3100 2600 50  0001 C CNN
+F 1 "GND" H 3105 2677 50  0000 C CNN
+F 2 "" H 3100 2850 50  0001 C CNN
+F 3 "" H 3100 2850 50  0001 C CNN
+	1    3100 2850
 	1    0    0    -1
 $EndComp
-Wire Wire Line
-	3100 2000 3100 2350
-Connection ~ 3100 2000
 Wire Wire Line
 	3650 2550 4600 2550
@@
 Wire Wire Line
 	5350 2250 5350 2200
+Wire Wire Line
+	2800 2300 3350 2300
+Wire Wire Line
+	2900 2650 2700 2650
+Wire Wire Line
+	3100 1700 3100 2450
+Wire Wire Line
+	2650 2200 2750 2200
+Wire Wire Line
+	2750 2200 2750 2450
+Wire Wire Line
+	2750 2450 3100 2450
+Connection ~ 3100 2450
+Wire Wire Line
+	3100 2450 3100 2550
+Wire Wire Line
+	2800 2000 2650 2000
+Wire Wire Line
+	2800 2000 2800 2300
+Wire Wire Line
+	2650 2300 2700 2300
+Wire Wire Line
+	2700 2300 2700 2650
 $EndSCHEMATC

Commit message: Update hum_temp_sensor.sch
Parts:
- R2: value 1k -> 220
Changed lines of the file:
@@
 P 5350 2050
 F 0 "R2" H 5420 2096 50  0000 L CNN
-F 1 "1k" H 5420 2005 50  0000 L CNN
+F 1 "220" H 5420 2005 50  0000 L CNN
 F 2 "Resistor_THT:R_Box_L13.0mm_W4.0mm_P9.00mm" V 5280 2050 50  0001 C CNN
 F 3 "~" H 5350 2050 50  0001 C CNN

Commit message: Update on 12V5A system power line
- 12V5A power line is now represented by two connectors with 2 pins across all the modules
- all .png previews are updated. The central hub now has previews for schematics, PCB tracing and 3D model
- peltier module now has two 12V5A connectors with redesigned one side of the bridge. Now all MOSFETs can be equipped with heatsinks
- hum/temp sensor now has its connector position reversed to mimic Grove's one
- hum/temp and gas sensors now have a small BeeHive logo on front layer rather than one big on back layer
- hum/temp sensor now use only one layer for signals and one layer for ground
- switch arrays now have two connectors for 12V5A and 5V3A power lines
- switch arrays had their power lines better traced (no sharp turns)
- power supply (12V5A to 5V3A) now has two connectors for 12V5A power line
- one trace of power supply, which lies in between LM2596's legs, was narrowed to ensure that it will not be accidentally soldered or damaged during placement
Changed lines of the file:
@@
 L power:GND #PWR01
 U 1 1 5F340F56
-P 2900 2650
-F 0 "#PWR01" H 2900 2400 50  0001 C CNN
-F 1 "GND" H 2905 2477 50  0000 C CNN
-F 2 "" H 2900 2650 50  0001 C CNN
-F 3 "" H 2900 2650 50  0001 C CNN
-	1    2900 2650
+P 2700 2850
+F 0 "#PWR01" H 2700 2600 50  0001 C CNN
+F 1 "GND" H 2705 2677 50  0000 C CNN
+F 2 "" H 2700 2850 50  0001 C CNN
+F 3 "" H 2700 2850 50  0001 C CNN
+	1    2700 2850
 	1    0    0    -1
 $EndComp
@@
 L power:GND #PWR08
 U 1 1 5F348437
-P 5350 2650
-F 0 "#PWR08" H 5350 2400 50  0001 C CNN
-F 1 "GND" H 5355 2477 50  0000 C CNN
-F 2 "" H 5350 2650 50  0001 C CNN
-F 3 "" H 5350 2650 50  0001 C CNN
-	1    5350 2650
+P 5350 2850
+F 0 "#PWR08" H 5350 2600 50  0001 C CNN
+F 1 "GND" H 5355 2677 50  0000 C CNN
+F 2 "" H 5350 2850 50  0001 C CNN
+F 3 "" H 5350 2850 50  0001 C CNN
+	1    5350 2850
 	1    0    0    -1
 $EndComp
 Wire Wire Line
-	5350 2650 5350 2550
+	5350 2850 5350 2550
 $Comp
 L Device:LED D1
@@
 Wire Wire Line
 	2800 2300 3350 2300
-Wire Wire Line
-	2900 2650 2700 2650
 Wire Wire Line
 	3100 1700 3100 2450
@@
 	2650 2300 2700 2300
 Wire Wire Line
-	2700 2300 2700 2650
+	2700 2300 2700 2850
 $EndSCHEMATC
