File: hardware/central_hub/beehive.kicad_pcb (KiCad board)
At the start: 2 copper layers, 76 x 85 mm, 30 parts, among them CON1 BARREL_JACK, P1 D1, P10 A2, P11 A3, P12 UART, P13 I2C 1, P14 I2C 2, P15 Conn_01x02, P16 Conn_01x02, P2 D2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

Commit message: Add an LED and 5V traces
Add LED to indicate that 12V power line is working
Edit 5V traces
Parts:
- added D2: LED, LED_THT:LED_D3.0mm, F.Cu at (206.5, 105.0)
- added R1: 560, Resistor_THT:R_Box_L13.0mm_W4.0mm_P9.00mm, F.Cu at (206.5, 112.5)
- moved C2 35.6 mm to (204.0, 84.5), turned to 270 degrees
- moved D1 21.9 mm to (192.0, 95.0), turned to 270 degrees
- moved   12.6 mm to (198.5, 79.5), turned to 0 degrees
- moved C1 11.2 mm to (196.0, 120.5), turned to 90 degrees
- moved L1 11.0 mm to (192.5, 89.5), turned to 90 degrees
- moved U1 6.02 mm to (200.5, 93.5)
- moved P11 2.00 mm to (180.5, 123.0)
- moved P10 1.00 mm to (170.5, 123.0)
Routing:
- net +5V: track 267.1 -> 288.9 mm, vias 1 -> 0
- net Net-(C1-Pad1): track 63.4 -> 74.8 mm
- net Net-(D1-Pad1): track 27.2 -> 20.5 mm
- net Net-(D2-Pad2): track 0.00 -> 4.96 mm
- net A3-3: track 33.0 -> 32.1 mm
- net A3-4: track 38.8 -> 38.3 mm
Other:
- board text added: "BeeHive v0.6"
- board text added: "POW"
- board text removed: "BeeHive v0.5"
