File: hardware/central_hub/beehive.sch (KiCad schematic (older format))
At the start: 23 parts, among them CON1 BARREL_JACK, P1 D1, P10 A2, P11 A3, P12 UART, P13 I2C 1, P14 I2C 2, P15 Conn_01x02, P16 Conn_01x02, P2 D2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

Commit message: Add an LED and 5V traces
Add LED to indicate that 12V power line is working
Edit 5V traces
Parts:
- added D2: LED, LED_THT:LED_D3.0mm, symbol Device:LED
- added R1: 560, Resistor_THT:R_Box_L13.0mm_W4.0mm_P9.00mm, symbol Device:R
Connections:
- net GND: now also D2.1 (K)
- net at C1.1, CON1.1, P15.1 (Pin_1)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: now also R1.2
- new net: D2.2 (A), R1.1
Changed lines of the file:
@@
 Main PS 5V3A
 Wire Wire Line
-	1550 2100 1550 5600
+	1550 2100 1550 3450
 $Comp
-L power:+5V #PWR?
+L power:+5V #PWR0111
 U 1 1 61EBF351
 P 10350 1950
-F 0 "#PWR?" H 10350 1800 50  0001 C CNN
+F 0 "#PWR0111" H 10350 1800 50  0001 C CNN
 F 1 "+5V" H 10350 2100 50  0000 C CNN
 F 2 "" H 10350 1950 50  0001 C CNN
@@
 	0    1    1    0
 $EndComp
+$Comp
+L Device:R R1
+U 1 1 61ED2F88
+P 2150 3450
+F 0 "R1" V 1943 3450 50  0000 C CNN
+F 1 "560" V 2034 3450 50  0000 C CNN
+F 2 "Resistor_THT:R_Box_L13.0mm_W4.0mm_P9.00mm" V 2080 3450 50  0001 C CNN
+F 3 "~" H 2150 3450 50  0001 C CNN
+	1    2150 3450
+	0    1    1    0
+$EndComp
+$Comp
+L Device:LED D2
+U 1 1 61ED3505
+P 2750 3450
+F 0 "D2" H 2743 3195 50  0000 C CNN
+F 1 "LED" H 2743 3286 50  0000 C CNN
+F 2 "LED_THT:LED_D3.0mm" H 2750 3450 50  0001 C CNN
+F 3 "~" H 2750 3450 50  0001 C CNN
+	1    2750 3450
+	-1   0    0    1
+$EndComp
+$Comp
+L power:GND #PWR0112
+U 1 1 61EDE164
+P 3300 3450
+F 0 "#PWR0112" H 3300 3200 50  0001 C CNN
+F 1 "GND" H 3300 3300 50  0000 C CNN
+F 2 "" H 3300 3450 50  0000 C CNN
+F 3 "" H 3300 3450 50  0000 C CNN
+	1    3300 3450
+	0    -1   -1   0
+$EndComp
+Wire Wire Line
+	1550 3450 2000 3450
+Connection ~ 1550 3450
+Wire Wire Line
+	1550 3450 1550 5600
+Wire Wire Line
+	2300 3450 2600 3450
+Wire Wire Line
+	2900 3450 3300 3450
 $EndSCHEMATC
