File: hardware/solenoid_driver/solenoid_driver.sch (KiCad schematic (older format))
At the start: 10 parts, among them J1 from_mainboard, J2 12V power, J3 to_solenoid2, J4 to_solenoid1, Q1 Q_NMOS_GDS, Q2 Q_NMOS_GDS

Commit message: cleanup of piezo amplifier and solenoid driver
Parts:
- J2, J3: footprint Connector_JST:JST_XH_B2B-XH-AM_1x02_P2.50mm_Vertical -> Connector_JST:JST_XH_B2B-XH-A_1x02_P2.50mm_Vertical
Changed lines of the file:
@@
 F 0 "J2" H 2722 5032 50  0000 R CNN
 F 1 "12V power" H 2722 5123 50  0000 R CNN
-F 2 "Connector_JST:JST_XH_B2B-XH-AM_1x02_P2.50mm_Vertical" H 2750 5150 50  0001 C CNN
+F 2 "Connector_JST:JST_XH_B2B-XH-A_1x02_P2.50mm_Vertical" H 2750 5150 50  0001 C CNN
 F 3 "~" H 2750 5150 50  0001 C CNN
 	1    2750 5150
@@
 F 0 "J3" H 7322 3024 50  0000 R CNN
 F 1 "to_solenoid2" H 7322 2933 50  0000 R CNN
-F 2 "Connector_JST:JST_XH_B2B-XH-AM_1x02_P2.50mm_Vertical" H 7350 3050 50  0001 C CNN
+F 2 "Connector_JST:JST_XH_B2B-XH-A_1x02_P2.50mm_Vertical" H 7350 3050 50  0001 C CNN
 F 3 "~" H 7350 3050 50  0001 C CNN
 	1    7350 3050
