File: hardware/solenoid_driver/_autosave-solenoid_driver.kicad_pcb (KiCad board)
At the start: 2 copper layers, 45.5 x 48.5 mm, 16 parts, among them J1 from_mainboard, J2 12V power, J3 to_solenoid2, J4 to_solenoid1, Q1 Q_NMOS_GDS, Q2 Q_NMOS_GDS

Commit message: update solenoid driver
Other:
- board text added: "board by Andre M Chagas licensed under CERN-OHL-S 2.0 https://ohwr.org/project/cernohl"
- board text removed: "board by Andre M Chagas licensed under CERN-OHL-W 2.0 https://ohwr.org/project/cernohl"
Changed lines of the file:
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@@
   (gr_line (start 157.5 80.5) (end 112 80.5) (layer "Edge.Cuts") (width 0.05))
   (gr_line (start 157.5 129) (end 112 129) (layer "Edge.Cuts") (width 0.05))
-  (gr_text "board by Andre M Chagas\nlicensed under\nCERN-OHL-W 2.0\nhttps://ohwr.org/project/cernohl" (at 139.7 124.714) (layer "F.SilkS")
+  (gr_text "board by Andre M Chagas\nlicensed under\nCERN-OHL-S 2.0\nhttps://ohwr.org/project/cernohl" (at 139.7 124.714) (layer "F.SilkS")
     (effects (font (size 0.75 0.75) (thickness 0.1)))
   )
