File: hardware/level_shifter/level_shifter.sch (KiCad schematic (older format))
At the start: 20 parts, among them J1 Conn_01x04, J2 Conn_01x04, J3 Conn_01x02, J4 Conn_01x02, J5 Conn_01x02, J6 Conn_01x02, Q1 2N7000, Q2 2N7000, Q3 2N7000, Q4 2N7000

Commit message: Add gerbers and screenshots
Added gerber files, screenshots and updated silkscreen
Other:
- note added: "3.25 V"
Changed lines of the file:
@@
 	1    0    0    -1
 $EndComp
+Text Notes 3200 1150 0    50   ~ 0
+3.25 V
 $EndSCHEMATC

Commit message: save the level shifter update also for the schematics
Parts:
- Q1, Q2, Q3, Q4: footprint Package_TO_SOT_THT:TO-92_Inline -> Package_TO_SOT_THT:TO-92_Inline_Wide
Changed lines of the file:
@@
 F 0 "Q1" V 5049 1450 50  0000 C CNN
 F 1 "2N7000" V 5140 1450 50  0000 C CNN
-F 2 "Package_TO_SOT_THT:TO-92_Inline" H 5000 1375 50  0001 L CIN
+F 2 "Package_TO_SOT_THT:TO-92_Inline_Wide" H 5000 1375 50  0001 L CIN
 F 3 "https://www.onsemi.com/pub/Collateral/NDS7002A-D.PDF" H 4800 1450 50  0001 L CNN
 	1    4800 1450
@@
 F 0 "Q2" V 5049 2550 50  0000 C CNN
 F 1 "2N7000" V 5140 2550 50  0000 C CNN
-F 2 "Package_TO_SOT_THT:TO-92_Inline" H 5000 2475 50  0001 L CIN
+F 2 "Package_TO_SOT_THT:TO-92_Inline_Wide" H 5000 2475 50  0001 L CIN
 F 3 "https://www.onsemi.com/pub/Collateral/NDS7002A-D.PDF" H 4800 2550 50  0001 L CNN
 	1    4800 2550
@@
 F 0 "Q3" V 5049 3600 50  0000 C CNN
 F 1 "2N7000" V 5140 3600 50  0000 C CNN
-F 2 "Package_TO_SOT_THT:TO-92_Inline" H 5000 3525 50  0001 L CIN
+F 2 "Package_TO_SOT_THT:TO-92_Inline_Wide" H 5000 3525 50  0001 L CIN
 F 3 "https://www.onsemi.com/pub/Collateral/NDS7002A-D.PDF" H 4800 3600 50  0001 L CNN
 	1    4800 3600
@@
 F 0 "Q4" V 5049 4750 50  0000 C CNN
 F 1 "2N7000" V 5140 4750 50  0000 C CNN
-F 2 "Package_TO_SOT_THT:TO-92_Inline" H 5000 4675 50  0001 L CIN
+F 2 "Package_TO_SOT_THT:TO-92_Inline_Wide" H 5000 4675 50  0001 L CIN
 F 3 "https://www.onsemi.com/pub/Collateral/NDS7002A-D.PDF" H 4800 4750 50  0001 L CNN
 	1    4800 4750
