File: hardware/testing_board/testing_board.kicad_sch (KiCad schematic)
At the start: 75 parts, among them J1 Conn_01x04, J16 Conn_01x04, J2 Conn_01x04, J3 Conn_01x04, J4 Conn_01x04, J5 Conn_01x04, J6 Conn_01x04, J7 Conn_01x04, J8 Conn_01x04, J9 Conn_01x04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

Commit message: work on training board updates
Other:
- note removed: "switch array"
Changed lines of the file:
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@@
-    (effects (font (size 1.27 1.27)) (justify left bottom))
-  )
-  (text "switch array" (at 86.36 69.85 0)
     (effects (font (size 1.27 1.27)) (justify left bottom))
   )
